File: FloppyEmulator.kicad_pcb (KiCad board)
At the start: 2 copper layers, 69.9 x 48.3 mm, 39 parts, among them Q1 Crystal_GND24, Q2 BC817, SW1 ALPS_5WAY, U1 STM32F405RGTx, U10 AP1117-15, U2 SN74LVC2G07, U3 SN74LVC2G07, U4 SN74LVC2G07, U5 SN74LVC2G07, U6 SN74LVC2G07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

Commit message: Backlight
Parts:
- added D1: LED_ALT, LEDs:LED_0805, F.Cu at (207.0, 81.9)
- added Q3: BC817, TO_SOT_Packages_SMD:SOT-23, F.Cu at (202.6, 81.9)
- added R2: 10K, Resistors_SMD:R_0603, F.Cu at (198.8, 80.6)
- added R3: 220, Resistors_SMD:R_0603, F.Cu at (199.4, 85.1)
- added R4: TBD, Resistors_SMD:R_0805, F.Cu at (144.8, 87.6)
Connections:
- U1 pad 25: /BUTTON1 -> /BUTTON3
- U1 pad 26: /BUTTON2 -> /BUTTON5
- U1 pad 27: /BUTTON3 -> /BUTTON2
- U1 pad 29: /BUTTON5 -> /BUTTON1
- U1 pad 54: /LCD_DC -> /LCD_RESET
- U1 pad 55: /LCD_RESET -> /LCD_DC
Routing:
- net +3V3: track 12.5 -> 138.0 mm, vias 7 -> 20
- net GND: track 18.4 -> 74.9 mm, vias 12 -> 27
- net /LED1: track 5.88 -> 56.3 mm
- net /BUTTON4: track 4.44 -> 38.5 mm
- net SPI2_MOSI: track 0.00 -> 31.2 mm, vias 0 -> 2
- net /BUTTON1: track 12.1 -> 43.2 mm
- net /BUTTON5: track 3.17 -> 33.7 mm
- net /BUTTON3: track 8.43 -> 35.4 mm
- net SPI3_MISO: track 0.00 -> 24.6 mm, vias 0 -> 1
- net SPI3_SCK: track 0.00 -> 22.9 mm, vias 0 -> 1
- net SPI3_MOSI: track 0.00 -> 21.5 mm, vias 0 -> 2
- net /BUTTON2: track 10.5 -> 31.9 mm
- net /LCD_DC: track 0.00 -> 19.6 mm
- net SPI3_NSS: track 0.00 -> 19.6 mm
- net /LCD_RESET: track 0.00 -> 19.3 mm
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- added copper zone on B.Cu, net +3V3
