File: FloppyEmulator.kicad_pcb (KiCad board)
At the start: 2 copper layers, 69.9 x 48.3 mm, 52 parts, among them Q1 Crystal_GND24, Q2 BC817, Q3 BC817, SW1 ALPS_5WAY, U1 STM32F405RGTx, U10 AP1117-15, U2 SN74LVC2G07, U3 SN74LVC2G07, U4 SN74LVC2G07, U5 SN74LVC2G07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

Commit message: Even more cleanups
Routing:
- net GND: track 390.6 -> 397.1 mm, vias 85 -> 88
- net /CARD_DETECT: track 39.7 -> 37.5 mm
- net /LED1: track 56.3 -> 57.4 mm
Changed lines of the file:
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@@
     (thickness 1.6)
     (drawings 10)
-    (tracks 682)
+    (tracks 687)
     (zones 0)
     (modules 52)
@@
   (segment (start 156.972 73.152) (end 157.405 73.585) (width 0.2) (layer F.Cu) (net 7))
   (segment (start 157.405 73.585) (end 161.305 73.585) (width 0.2) (layer F.Cu) (net 7))
+  (segment (start 187.198 68.834) (end 183.896 68.834) (width 0.2) (layer B.Cu) (net 8))
+  (segment (start 183.896 68.834) (end 183.642 69.088) (width 0.2) (layer B.Cu) (net 8))
+  (via (at 183.642 69.088) (size 0.9) (drill 0.4) (layers F.Cu B.Cu) (net 8))
+  (segment (start 200.152 61.976) (end 191.008 61.976) (width 0.2) (layer F.Cu) (net 8))
+  (segment (start 200.914 62.738) (end 200.152 61.976) (width 0.2) (layer F.Cu) (net 8))
+  (via (at 191.008 61.976) (size 0.9) (drill 0.4) (layers F.Cu B.Cu) (net 8))
+  (segment (start 191.008 65.278) (end 187.452 68.834) (width 0.2) (layer F.Cu) (net 8))
+  (segment (start 187.452 68.834) (end 187.198 68.834) (width 0.2) (layer F.Cu) (net 8))
+  (via (at 187.198 68.834) (size 0.9) (drill 0.4) (layers F.Cu B.Cu) (net 8))
+  (segment (start 202.692 60.96) (end 200.914 62.738) (width 0.5) (layer B.Cu) (net 8))
+  (segment (start 203.2 60.96) (end 202.692 60.96) (width 0.5) (layer B.Cu) (net 8))
+  (via (at 200.914 62.738) (size 0.9) (drill 0.4) (layers F.Cu B.Cu) (net 8))
+  (segment (start 201.93 67.945) (end 198.247 64.262) (width 0.5) (layer B.Cu) (net 8))
+  (segment (start 198.247 64.262) (end 197.866 64.262) (width 0.5) (layer B.Cu) (net 8))
+  (segment (start 197.416001 64.711999) (end 197.866 64.262) (width 0.2) (layer F.Cu) (net 8))
+  (segment (start 196.85 65.278) (end 197.416001 64.711999) (width 0.2) (layer F.Cu) (net 8))
+  (segment (start 196.85 73.66) (end 196.85 65.278) (width 0.2) (layer F.Cu) (net 8))
+  (via (at 197.866 64.262) (size 0.9) (drill 0.4) (layers F.Cu B.Cu) (net 8))
   (segment (start 201.93 67.945) (end 205.105 67.945) (width 0.5) (layer B.Cu) (net 8))
   (via (at 205.105 67.945) (size 0.9) (drill 0.4) (layers F.Cu B.Cu) (net 8))
-  (segment (start 201.295 67.945) (end 201.93 67.945) (width 0.5) (layer B.Cu) (net 8))
-  (segment (start 196.85 63.5) (end 201.295 67.945) (width 0.5) (layer B.Cu) (net 8))
   (via (at 201.93 67.945) (size 0.9) (drill 0.4) (layers F.Cu B.Cu) (net 8))
   (segment (start 163.576 76.454) (end 163.576 74.954) (width 1) (layer B.Cu) (net 8))
@@
   (segment (start 191.12 65.39) (end 191.008 65.278) (width 0.5) (layer F.Cu) (net 8))
   (segment (start 190.371604 65.278) (end 191.008 65.278) (width 0.2) (layer B.Cu) (net 8))
-  (segment (start 190.246 65.278) (end 190.371604 65.278) (width 0.2) (layer F.Cu) (net 8))
-  (segment (start 190.371604 65.278) (end 191.008 65.278) (width 0.2) (layer F.Cu) (net 8))
   (segment (start 192.69 65.39) (end 191.12 65.39) (width 0.5) (layer F.Cu) (net 8))
   (segment (start 187.198 65.278) (end 190.371604 65.278) (width 0.2) (layer B.Cu) (net 8))
-  (segment (start 186.69 68.834) (end 190.246 65.278) (width 0.2) (layer F.Cu) (net 8))
   (segment (start 191.644396 65.278) (end 191.008 65.278) (width 0.2) (layer B.Cu) (net 8))
   (segment (start 191.516 65.278) (end 191.008 65.278) (width 0.5) (layer F.Cu) (net 8))
   (segment (start 191.628 65.39) (end 191.516 65.278) (width 0.5) (layer F.Cu) (net 8))
   (via (at 191.008 65.278) (size 0.9) (drill 0.4) (layers F.Cu B.Cu) (net 8))
-  (via (at 186.69 68.834) (size 0.9) (drill 0.4) (layers F.Cu B.Cu) (net 8))
   (segment (start 174.625 86.487) (end 172.974 84.836) (width 0.2) (layer F.Cu) (net 8))
   (segment (start 174.625 87.63) (end 174.625 86.487) (width 0.2) (layer F.Cu) (net 8))
@@
   (segment (start 192.69 78.04) (end 192.69 79.66) (width 0.2) (layer F.Cu) (net 8))
   (via (at 193.04 80.01) (size 0.9) (drill 0.4) (layers F.Cu B.Cu) (net 8))
-  (segment (start 198.12 72.39) (end 196.85 73.66) (width 0.2) (layer F.Cu) (net 8))
-  (segment (start 198.12 69.85) (end 198.12 72.39) (width 0.2) (layer F.Cu) (net 8))
   (via (at 196.85 73.66) (size 0.9) (drill 0.4) (layers F.Cu B.Cu) (net 8))
-  (segment (start 199.39 71.12) (end 198.12 69.85) (width 0.2) (layer F.Cu) (net 8))
-  (segment (start 201.93 71.12) (end 199.39 71.12) (width 0.2) (layer F.Cu) (net 8))
-  (segment (start 199.39 68.58) (end 201.93 71.12) (width 0.2) (layer F.Cu) (net 8))
-  (segment (start 199.39 66.04) (end 199.39 68.58) (width 0.2) (layer F.Cu) (net 8))
-  (segment (start 199.39 66.04) (end 196.85 63.5) (width 0.2) (layer F.Cu) (net 8))
-  (via (at 196.85 63.5) (size 0.9) (drill 0.4) (layers F.Cu B.Cu) (net 8))
   (segment (start 194.408 68.99) (end 194.564 68.834) (width 0.2) (layer F.Cu) (net 8))
   (segment (start 192.79 68.99) (end 194.408 68.99) (width 0.2) (layer F.Cu) (net 8))
@@
   (segment (start 199.009 80.264) (end 190.373 71.628) (width 0.2) (layer B.Cu) (net 15))
   (segment (start 184.024398 71.628) (end 183.388002 71.628) (width 0.2) (layer B.Cu) (net 15))
-  (segment (start 195.58 63.5) (end 195.58 70.612) (width 0.2) (layer F.Cu) (net 28))
-  (segment (start 190.246 63.5) (end 195.58 63.5) (width 0.2) (layer F.Cu) (net 28))
-  (segment (start 184.912 68.834) (end 190.246 63.5) (width 0.2) (layer F.Cu) (net 28))
-  (segment (start 184.912 72.898) (end 184.912 68.834) (width 0.2) (layer F.Cu) (net 28))
-  (segment (start 180.225 77.585) (end 184.912 72.898) (width 0.2) (layer F.Cu) (net 28))
+  (segment (start 191.008 63.5) (end 195.326 63.5) (width 0.2) (layer F.Cu) (net 28))
+  (segment (start 185.166 69.342) (end 191.008 63.5) (width 0.2) (layer F.Cu) (net 28))
+  (segment (start 180.225 77.585) (end 185.166 72.644) (width 0.2) (layer F.Cu) (net 28))
+  (segment (start 196.088 70.104) (end 193.902 72.29) (width 0.2) (layer F.Cu) (net 28))
+  (segment (start 185.166 72.644) (end 185.166 69.342) (width 0.2) (layer F.Cu) (net 28))
   (segment (start 172.705 77.585) (end 180.225 77.585) (width 0.2) (layer F.Cu) (net 28))
-  (segment (start 195.58 70.612) (end 193.902 72.29) (width 0.2) (layer F.Cu) (net 28))
+  (segment (start 195.326 63.5) (end 196.088 64.262) (width 0.2) (layer F.Cu) (net 28))
+  (segment (start 196.088 64.262) (end 196.088 70.104) (width 0.2) (layer F.Cu) (net 28))
   (segment (start 193.902 72.29) (end 192.79 72.29) (width 0.2) (layer F.Cu) (net 28))
   (segment (start 180.487 78.085) (end 188.595 69.977) (width 0.2) (layer F.Cu) (net 29))
@@
   (segment (start 151.13 81.28) (end 151.892 80.518) (width 0.2) (layer F.Cu) (net 39))
   (segment (start 146.37 94.15) (end 146.37 86.04) (width 0.2) (layer F.Cu) (net 39))
-  (segment (start 179.963 77.085) (end 184.404 72.644) (width 0.2) (layer F.Cu) (net 48))
+  (segment (start 198.628 62.992) (end 200.376 64.74) (width 0.2) (layer F.Cu) (net 48))
+  (segment (start 184.658 69.088) (end 190.754 62.992) (width 0.2) (layer F.Cu) (net 48))
+  (segment (start 184.658 72.39) (end 184.658 69.088) (width 0.2) (layer F.Cu) (net 48))
+  (segment (start 200.376 64.74) (end 201.74 64.74) (width 0.2) (layer F.Cu) (net 48))
   (segment (start 172.705 77.085) (end 179.963 77.085) (width 0.2) (layer F.Cu) (net 48))
-  (segment (start 191.008 61.976) (end 200.406 61.976) (width 0.2) (layer F.Cu) (net 48))
-  (segment (start 184.404 72.644) (end 184.404 68.58) (width 0.2) (layer F.Cu) (net 48))
-  (segment (start 184.404 68.58) (end 191.008 61.976) (width 0.2) (layer F.Cu) (net 48))
-  (segment (start 201.74 63.31) (end 201.74 64.74) (width 0.2) (layer F.Cu) (net 48))
-  (segment (start 200.406 61.976) (end 201.74 63.31) (width 0.2) (layer F.Cu) (net 48))
+  (segment (start 190.754 62.992) (end 198.628 62.992) (width 0.2) (layer F.Cu) (net 48))
+  (segment (start 179.963 77.085) (end 184.658 72.39) (width 0.2) (layer F.Cu) (net 48))
   (segment (start 182.245 98.425) (end 180.975 98.425) (width 0.25) (layer B.Cu) (net 69))
   (segment (start 184.15 100.33) (end 182.245 98.425) (width 0.25) (layer B.Cu) (net 69))
@@
   (segment (start 175.018 73.14) (end 175.018 72.39) (width 0.25) (layer F.Cu) (net 82))
   (segment (start 172.705 73.585) (end 174.573 73.585) (width 0.25) (layer F.Cu) (net 82))
-  (segment (start 203.835 64.135) (end 203.835 71.12) (width 0.2) (layer F.Cu) (net 83))
-  (segment (start 172.705 74.085) (end 177.375 74.085) (width 0.2) (layer F.Cu) (net 83))
+  (segment (start 204.216 64.008) (end 204.216 70.739) (width 0.2) (layer F.Cu) (net 83))
+  (segment (start 190.5 60.96) (end 201.168 60.96) (width 0.2) (layer F.Cu) (net 83))
   (segment (start 198.005 76.95) (end 198.005 79.995) (width 0.2) (layer F.Cu) (net 83))
-  (segment (start 201.27599 61.57599) (end 203.835 64.135) (width 0.2) (layer F.Cu) (net 83))
-  (segment (start 203.835 71.12) (end 198.005 76.95) (width 0.2) (layer F.Cu) (net 83))
-  (segment (start 189.88401 61.57599) (end 201.27599 61.57599) (width 0.2) (layer F.Cu) (net 83))
-  (segment (start 177.375 74.085) (end 189.88401 61.57599) (width 0.2) (layer F.Cu) (net 83))
+  (segment (start 204.216 70.739) (end 198.005 76.95) (width 0.2) (layer F.Cu) (net 83))
   (segment (start 198.005 79.995) (end 198.005 80.645) (width 0.2) (layer F.Cu) (net 83))
+  (segment (start 201.168 60.96) (end 204.216 64.008) (width 0.2) (layer F.Cu) (net 83))
+  (segment (start 172.705 74.085) (end 177.375 74.085) (width 0.2) (layer F.Cu) (net 83))
+  (segment (start 177.375 74.085) (end 190.5 60.96) (width 0.2) (layer F.Cu) (net 83))
   (segment (start 152.4 96.35) (end 152.4 97.198998) (width 0.2) (layer F.Cu) (net 84))
   (segment (start 152.4 97.198998) (end 152.374998 97.224) (width 0.2) (layer F.Cu) (net 84))
