File: FloppyEmulator.kicad_pcb (KiCad board)
At the start: 2 copper layers, 67.4 x 48.3 mm, 52 parts, among them Q1 Crystal_GND24, Q2 BC817, Q3 BC817, SW1 ALPS_5WAY, U1 STM32F405RGTx, U10 AP1117-15, U2 SN74LVC2G07, U3 SN74LVC2G07, U4 SN74LVC2G07, U5 SN74LVC2G07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

Commit message: More final touches
Parts:
- moved C17 0.51 mm to (182.9, 94.7)
- moved C18 0.51 mm to (177.8, 94.7)
Routing:
- net GND: track 325.8 -> 342.1 mm, vias 83 -> 84
- net (no net): vias 2 -> 1
Changed lines of the file:
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@@
-(kicad_pcb (version 20171130) (host pcbnew no-vcs-found-e062780~61~ubuntu17.10.1)
+(kicad_pcb (version 20171130) (host pcbnew no-vcs-found-bf44d39~61~ubuntu17.10.1)
   (general
     (thickness 1.6)
     (drawings 10)
-    (tracks 662)
+    (tracks 666)
     (zones 0)
     (modules 52)
@@
   )
   (setup
-    (last_trace_width 0.5)
+    (last_trace_width 0.2)
     (user_trace_width 0.2)
     (user_trace_width 0.25)
@@
   (module QVGA_LCD_9pin (layer F.Cu)
     (at 144.78 77.47 270)
-    (fp_text reference X2 (at 2.54 -9.66 270) (layer F.SilkS)
+    (fp_text reference X2 (at 0 -2.54 270) (layer F.SilkS)
       (effects (font (size 1 1) (thickness 0.15)))
     )
@@
     (descr "Crystal THT HC-49/U http://5hertz.com/pdfs/04404_D.pdf")
     (tags "THT crystalHC-49/U")
-    (fp_text reference Q1 (at 2.44 -3.525 180) (layer F.SilkS)
+    (fp_text reference Q1 (at 2.286 -0.127 180) (layer F.SilkS)
       (effects (font (size 1 1) (thickness 0.15)))
     )
@@
     (descr "Through hole straight pin header, 1x04, 2.54mm pitch, single row")
     (tags "Through hole pin header THT 1x04 2.54mm single row")
-    (fp_text reference X5 (at 0 -2.33 90) (layer F.SilkS)
+    (fp_text reference X5 (at 0 -2.33 180) (layer F.SilkS)
       (effects (font (size 1 1) (thickness 0.15)))
     )
@@
   (module components:MOLEX_5027740891 locked (layer F.Cu)
     (at 200.66 71.12 90)
-    (fp_text reference X1 (at 13 0.5 90) (layer F.SilkS)
+    (fp_text reference X1 (at 0 0.5) (layer F.SilkS)
       (effects (font (size 1 1) (thickness 0.15)))
     )
@@
     (tags "QFP 0.5")
     (attr smd)
-    (fp_text reference U1 (at 0 -7.2 90) (layer F.SilkS)
+    (fp_text reference U1 (at 0.127 -0.127 180) (layer F.SilkS)
       (effects (font (size 1 1) (thickness 0.15)))
     )
@@
     (tags SOT-23-6)
     (attr smd)
-    (fp_text reference U2 (at 0 -2.9 90) (layer F.SilkS)
+    (fp_text reference U2 (at 0 0 180) (layer F.SilkS)
       (effects (font (size 1 1) (thickness 0.15)))
     )
@@
     (tags SOT-23-6)
     (attr smd)
-    (fp_text reference U3 (at 0 -2.9 90) (layer F.SilkS)
+    (fp_text reference U3 (at 0 0 180) (layer F.SilkS)
       (effects (font (size 1 1) (thickness 0.15)))
     )
@@
     (tags SOT-23-6)
     (attr smd)
-    (fp_text reference U4 (at 0 -2.9 90) (layer F.SilkS)
+    (fp_text reference U4 (at 0 0 180) (layer F.SilkS)
       (effects (font (size 1 1) (thickness 0.15)))
     )
@@
     (tags SOT-23-6)
     (attr smd)
-    (fp_text reference U5 (at 0 -2.9 90) (layer F.SilkS)
+    (fp_text reference U5 (at 0 0 180) (layer F.SilkS)
       (effects (font (size 1 1) (thickness 0.15)))
     )
@@
     (tags SOT-23-6)
     (attr smd)
-    (fp_text reference U6 (at 0 -2.9 270) (layer F.SilkS)
+    (fp_text reference U6 (at 0 -0.254) (layer F.SilkS)
       (effects (font (size 1 1) (thickness 0.15)))
     )
@@
     (tags SOT-23-6)
     (attr smd)
-    (fp_text reference U7 (at 0 -2.9 270) (layer F.SilkS)
+    (fp_text reference U7 (at 0 0) (layer F.SilkS)
       (effects (font (size 1 1) (thickness 0.15)))
     )
@@
     (tags SOT-23-6)
     (attr smd)
-    (fp_text reference U8 (at 0 -2.9 90) (layer F.SilkS)
+    (fp_text reference U8 (at 0 0 180) (layer F.SilkS)
       (effects (font (size 1 1) (thickness 0.15)))
     )
@@
     (tags SOT-23-6)
     (attr smd)
-    (fp_text reference U9 (at 0 -2.9 270) (layer F.SilkS)
+    (fp_text reference U9 (at 0 0) (layer F.SilkS)
       (effects (font (size 1 1) (thickness 0.15)))
     )
@@
     (tags "resistor 0603")
     (attr smd)
-    (fp_text reference R1 (at 0 -1.45 270) (layer F.SilkS)
+    (fp_text reference R1 (at 0.012 1.397 270) (layer F.SilkS)
       (effects (font (size 1 1) (thickness 0.15)))
     )
@@
     (tags "capacitor 0805")
     (attr smd)
-    (fp_text reference C6 (at 0 -1.5 90) (layer F.SilkS)
+    (fp_text reference C6 (at 0 1.778 90) (layer F.SilkS)
       (effects (font (size 1 1) (thickness 0.15)))
     )
@@
     (tags "capacitor 0805")
     (attr smd)
-    (fp_text reference C7 (at 0 -1.5 270) (layer F.SilkS)
+    (fp_text reference C7 (at 0 1.524 270) (layer F.SilkS)
       (effects (font (size 1 1) (thickness 0.15)))
     )
@@
     (tags "CMS SOT")
     (attr smd)
-    (fp_text reference U10 (at 0 -4.5 90) (layer F.SilkS)
+    (fp_text reference U10 (at -0.508 0 180) (layer F.SilkS)
       (effects (font (size 1 1) (thickness 0.15)))
     )
@@
   )
   (module Capacitors_SMD:C_0603 (layer B.Cu)
-    (at 182.88 95.25 90)
+    (at 182.88 94.742 90)
     (descr "Capacitor SMD 0603, reflow soldering, AVX (see smccp.pdf)")
     (tags "capacitor 0603")
@@
   )
   (module Capacitors_SMD:C_0603 (layer B.Cu)
-    (at 177.8 95.25 90)
+    (at 177.8 94.742 90)
     (descr "Capacitor SMD 0603, reflow soldering, AVX (see smccp.pdf)")
     (tags "capacitor 0603")
@@
     (tags SOT-23)
     (attr smd)
-    (fp_text reference Q3 (at 0 -2.5) (layer F.SilkS)
+    (fp_text reference Q3 (at 0.127 2.413) (layer F.SilkS)
       (effects (font (size 1 1) (thickness 0.15)))
     )
@@
   (module components:HCM1206A (layer F.Cu)
     (at 178.435 64.135 270)
-    (fp_text reference BA1 (at 0 2.75 270) (layer F.SilkS)
+    (fp_text reference BA1 (at 0.635 -0.635) (layer F.SilkS)
       (effects (font (size 1 1) (thickness 0.15)))
     )
@@
     (tags "capacitor 0805")
     (attr smd)
-    (fp_text reference C14 (at 0 -1.5 180) (layer F.SilkS)
+    (fp_text reference C14 (at 0 1.524 180) (layer F.SilkS)
       (effects (font (size 1 1) (thickness 0.15)))
     )
@@
     (tags "resistor 0603")
     (attr smd)
-    (fp_text reference R5 (at 0 -1.45 180) (layer F.SilkS)
+    (fp_text reference R5 (at 0 1.524 180) (layer F.SilkS)
       (effects (font (size 1 1) (thickness 0.15)))
     )
@@
     (tags "resistor 0603")
     (attr smd)
-    (fp_text reference R6 (at 0 -1.45 270) (layer F.SilkS)
+    (fp_text reference R6 (at 0 1.397 270) (layer F.SilkS)
       (effects (font (size 1 1) (thickness 0.15)))
     )
@@
   (segment (start 157.556704 73.585) (end 160.605 73.585) (width 0.2) (layer F.Cu) (net 7))
   (segment (start 160.605 73.585) (end 161.305 73.585) (width 0.2) (layer F.Cu) (net 7))
+  (segment (start 152.146 58.674) (end 148.59 62.23) (width 0.5) (layer B.Cu) (net 8))
+  (segment (start 161.036 58.674) (end 152.146 58.674) (width 0.5) (layer B.Cu) (net 8))
+  (via (at 148.59 62.23) (size 0.9) (drill 0.4) (layers F.Cu B.Cu) (net 8))
+  (segment (start 161.29 58.928) (end 161.036 58.674) (width 0.5) (layer B.Cu) (net 8))
+  (segment (start 161.29 60.96) (end 161.29 58.928) (width 0.5) (layer B.Cu) (net 8))
   (segment (start 148.59 76.2) (end 151.13 76.2) (width 0.2) (layer F.Cu) (net 8))
   (via (at 151.13 76.2) (size 0.9) (drill 0.4) (layers F.Cu B.Cu) (net 8))
@@
   (via (at 187.96 60.96) (size 0.9) (drill 0.4) (layers F.Cu B.Cu) (net 8))
   (via (at 182.88 60.96) (size 0.9) (drill 0.4) (layers F.Cu B.Cu) (net 8))
-  (via (at 152.4 60.96) (size 0.9) (drill 0.4) (layers F.Cu B.Cu) (net 0))
   (segment (start 161.29 60.96) (end 158.75 58.42) (width 0.2) (layer B.Cu) (net 8))
   (segment (start 170.18 98.425) (end 175.26 98.425) (width 0.2) (layer B.Cu) (net 8))
