File: FloppyEmulator.sch (KiCad schematic (older format))
At the start: 37 parts, among them Q1 Crystal_GND24, Q2 BC817, SW1 ALPS_5WAY, U1 STM32F405RGTx, U10 AP1117-15, U2 SN74LVC2G07, U3 SN74LVC2G07, U4 SN74LVC2G07, U5 SN74LVC2G07, U6 SN74LVC2G07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

Commit message: Routing WIP
Parts:
- added C? (x2): 15pF, Capacitors_SMD:C_0603, symbol device1:C
Connections:
- wire segments 261 -> 264
Changed lines of the file:
@@
 Wire Wire Line
 	12875 6000 13175 6000
+$Comp
+L device1:C C?
+U 1 1 5A64000B
+P 3350 4500
+F 0 "C?" H 3465 4546 50  0000 L CNN
+F 1 "15pF" H 3465 4455 50  0000 L CNN
+F 2 "Capacitors_SMD:C_0603" H 3388 4350 50  0001 C CNN
+F 3 "" H 3350 4500 50  0001 C CNN
+	1    3350 4500
+	0    -1   -1   0
+$EndComp
+$Comp
+L device1:C C?
+U 1 1 5A6402DE
+P 3350 4950
+F 0 "C?" H 3465 4996 50  0000 L CNN
+F 1 "15pF" H 3465 4905 50  0000 L CNN
+F 2 "Capacitors_SMD:C_0603" H 3388 4800 50  0001 C CNN
+F 3 "" H 3350 4950 50  0001 C CNN
+	1    3350 4950
+	0    -1   -1   0
+$EndComp
+Wire Wire Line
+	3500 4950 3650 4950
+Connection ~ 3650 4950
+Wire Wire Line
+	3500 4500 3725 4500
+Wire Wire Line
+	3725 4500 3725 4550
+Connection ~ 3725 4550
+$Comp
+L power1:GND #PWR?
+U 1 1 5A66A249
+P 3200 4500
+F 0 "#PWR?" H 3200 4250 50  0001 C CNN
+F 1 "GND" H 3205 4327 50  0001 C CNN
+F 2 "" H 3200 4500 50  0001 C CNN
+F 3 "" H 3200 4500 50  0001 C CNN
+	1    3200 4500
+	0    1    -1   0
+$EndComp
+$Comp
+L power1:GND #PWR?
+U 1 1 5A66A2F0
+P 3200 4950
+F 0 "#PWR?" H 3200 4700 50  0001 C CNN
+F 1 "GND" H 3205 4777 50  0001 C CNN
+F 2 "" H 3200 4950 50  0001 C CNN
+F 3 "" H 3200 4950 50  0001 C CNN
+	1    3200 4950
+	0    1    -1   0
+$EndComp
 $EndSCHEMATC

Commit message: Backlight
Parts:
- added D1: LED_ALT, LEDs:LED_0805, symbol device1:LED_ALT
- added Q3: BC817, TO_SOT_Packages_SMD:SOT-23, symbol device1:Q_NPN_BEC
- added R2: 10K, Resistors_SMD:R_0603, symbol device1:R
- added R3: 220, Resistors_SMD:R_0603, symbol device1:R
- added R?: TBD, Resistors_SMD:R_0805, symbol device1:R
- gave numbers to parts that had none: 2
Connections:
- wire segments 264 -> 268

Commit message: Copper pours
Parts:
- removed C14, C15: 0,1, Capacitors_SMD:C_0603, symbol device1:C
- gave numbers to parts that had none: 1
Connections:
- wire segments 268 -> 260
Changed lines of the file:
@@
-	1    0    0    -1
-$EndComp
-$Comp
-L device1:C C14
-U 1 1 5A5B3AD8
-P 13175 2625
-F 0 "C14" H 13290 2671 50  0000 L CNN
-F 1 "0,1" H 13290 2580 50  0000 L CNN
-F 2 "Capacitors_SMD:C_0603" H 13213 2475 50  0001 C CNN
-F 3 "" H 13175 2625 50  0001 C CNN
-	1    13175 2625
-	1    0    0    -1
-$EndComp
-$Comp
-L device1:C C15
-U 1 1 5A5B3ADE
-P 13525 2625
-F 0 "C15" H 13640 2671 50  0000 L CNN
-F 1 "0,1" H 13640 2580 50  0000 L CNN
-F 2 "Capacitors_SMD:C_0603" H 13563 2475 50  0001 C CNN
-F 3 "" H 13525 2625 50  0001 C CNN
-	1    13525 2625
 	1    0    0    -1
 $EndComp
 Wire Wire Line
 	12075 2325 12450 2325
-Wire Wire Line
-	13525 2325 13525 2475
-Wire Wire Line
-	13525 2775 13525 2850
-Wire Wire Line
-	13525 2850 13175 2850
 Wire Wire Line
 	12450 2475 12450 2325
@@
 Wire Wire Line
 	12825 2475 12825 2325
-Connection ~ 12825 2325
-Wire Wire Line
-	12825 2325 13175 2325
-Wire Wire Line
-	13175 2475 13175 2325
-Connection ~ 13175 2325
-Wire Wire Line
-	13175 2325 13525 2325
 Wire Wire Line
 	12450 2775 12450 2850
@@
 Wire Wire Line
 	12825 2775 12825 2850
-Connection ~ 12825 2850
 Wire Wire Line
 	12825 2850 12450 2850
-Wire Wire Line
-	13175 2775 13175 2850
-Connection ~ 13175 2850
-Wire Wire Line
-	13175 2850 12825 2850
 Connection ~ 12075 2325
 Connection ~ 12075 2850
@@
 +5VDC
 $Comp
-L device1:R R?
+L device1:R R4
 U 1 1 5A701DF4
 P 1325 7075
-F 0 "R?" V 1118 7075 50  0000 C CNN
+F 0 "R4" V 1118 7075 50  0000 C CNN
 F 1 "TBD" V 1209 7075 50  0000 C CNN
 F 2 "Resistors_SMD:R_0805" V 1255 7075 50  0001 C CNN

Commit message: Add HCM1206A beeper
Parts:
- added BA1: HCM1206A, components:HCM1206A, symbol device1:Speaker
- added C?: 2u2, Capacitors_SMD:C_0805, symbol device1:C
- added R5: TBD, Resistors_SMD:R_0603, symbol device1:R
Connections:
- wire segments 260 -> 268
Changed lines of the file:
@@
 Wire Wire Line
 	1850 7075 1475 7075
+$Comp
+L device1:Speaker BA1
+U 1 1 5A7572E3
+P 15425 3900
+F 0 "BA1" H 15595 3896 50  0000 L CNN
+F 1 "HCM1206A" H 15595 3805 50  0000 L CNN
+F 2 "components:HCM1206A" H 15425 3700 50  0001 C CNN
+F 3 "" H 15415 3850 50  0001 C CNN
+	1    15425 3900
+	1    0    0    -1
+$EndComp
+$Comp
+L device1:R R5
+U 1 1 5A75742F
+P 15150 3625
+F 0 "R5" V 14943 3625 50  0000 C CNN
+F 1 "TBD" V 15034 3625 50  0000 C CNN
+F 2 "Resistors_SMD:R_0603" V 15080 3625 50  0001 C CNN
+F 3 "" H 15150 3625 50  0001 C CNN
+	1    15150 3625
+	-1   0    0    1
+$EndComp
+Wire Wire Line
+	15150 3775 15150 3900
+Wire Wire Line
+	15150 3900 15225 3900
+Wire Wire Line
+	15225 4000 15150 4000
+Wire Wire Line
+	15150 4000 15150 4200
+Text GLabel 14575 3325 0    60   Input ~ 0
++3V3
+Wire Wire Line
+	14575 3325 14800 3325
+Wire Wire Line
+	15150 3325 15150 3475
+$Comp
+L device1:C C?
+U 1 1 5A7ABDC3
+P 14800 3625
+F 0 "C?" H 14915 3671 50  0000 L CNN
+F 1 "2u2" H 14915 3580 50  0000 L CNN
+F 2 "Capacitors_SMD:C_0805" H 14838 3475 50  0001 C CNN
+F 3 "" H 14800 3625 50  0001 C CNN
+	1    14800 3625
+	1    0    0    -1
+$EndComp
+$Comp
+L power1:GND #PWR?
+U 1 1 5A7ABFFF
+P 14800 3775
+F 0 "#PWR?" H 14800 3525 50  0001 C CNN
+F 1 "GND" H 14805 3602 50  0001 C CNN
+F 2 "" H 14800 3775 50  0001 C CNN
+F 3 "" H 14800 3775 50  0001 C CNN
+	1    14800 3775
+	1    0    0    -1
+$EndComp
+Wire Wire Line
+	14800 3475 14800 3325
+Connection ~ 14800 3325
+Wire Wire Line
+	14800 3325 15150 3325
 $EndSCHEMATC

Commit message: Add I2C
Parts:
- added C15, C? (x2): 0,1, Capacitors_SMD:C_0603, symbol device1:C
- gave numbers to parts that had none: 1
Connections:
- wire segments 268 -> 271
Changed lines of the file:
@@
 Text GLabel 13100 6200 2    50   BiDi ~ 0
 SDA
-Text Notes 850  3825 0    60   ~ 0
+Text Notes 775  5025 0    60   ~ 0
 BUTTONS, LED(s) and BEEPER
 Text Notes 13700 6675 0    60   ~ 0
@@
 Text Notes 12450 1325 0    60   ~ 0
 ESD?\nPull-ups?
-Text Notes 825  4075 0    60   ~ 0
+Text Notes 750  5275 0    60   ~ 0
 SN74LV1T34 Logic Buffer Translator\nSN74LVC2G07 Dual Open Drain Buffer
 $Comp
@@
 Text Label 13650 6400 2    60   ~ 0
 LED1
-Wire Wire Line
-	4275 4000 3800 4000
 Text Label 3800 4000 0    60   ~ 0
 VBAT
@@
 	15150 3325 15150 3475
 $Comp
-L device1:C C?
+L device1:C C14
 U 1 1 5A7ABDC3
 P 14800 3625
-F 0 "C?" H 14915 3671 50  0000 L CNN
+F 0 "C14" H 14915 3671 50  0000 L CNN
 F 1 "2u2" H 14915 3580 50  0000 L CNN
 F 2 "Capacitors_SMD:C_0805" H 14838 3475 50  0001 C CNN
@@
 $EndComp
 $Comp
-L power1:GND #PWR?
+L power1:GND #PWR032
 U 1 1 5A7ABFFF
 P 14800 3775
-F 0 "#PWR?" H 14800 3525 50  0001 C CNN
+F 0 "#PWR032" H 14800 3525 50  0001 C CNN
 F 1 "GND" H 14805 3602 50  0001 C CNN
 F 2 "" H 14800 3775 50  0001 C CNN
@@
 Wire Wire Line
 	14800 3325 15150 3325
+$Comp
+L device1:C C15
+U 1 1 5A7D76FB
+P 3250 3875
+F 0 "C15" H 3365 3921 50  0000 L CNN
+F 1 "0,1" H 3365 3830 50  0000 L CNN
+F 2 "Capacitors_SMD:C_0603" H 3288 3725 50  0001 C CNN
+F 3 "" H 3250 3875 50  0001 C CNN
+	1    3250 3875
+	-1   0    0    1
+$EndComp
+$Comp
+L power1:GND #PWR033
+U 1 1 5A7D78C7
+P 3250 4025
+F 0 "#PWR033" H 3250 3775 50  0001 C CNN
+F 1 "GND" H 3255 3852 50  0001 C CNN
+F 2 "" H 3250 4025 50  0001 C CNN
+F 3 "" H 3250 4025 50  0001 C CNN
+	1    3250 4025
+	-1   0    0    -1
+$EndComp
+Wire Wire Line
+	3550 4000 3550 3725
+Wire Wire Line
+	3550 3725 3250 3725
+Wire Wire Line
+	3550 4000 4275 4000
+Wire Wire Line
+	3250 3725 2925 3725
+Connection ~ 3250 3725
+Text GLabel 2925 3725 0    60   Input ~ 0
++3V3
+$Comp
+L device1:C C?
+U 1 1 5A819C2F
+P 1250 3950
+F 0 "C?" H 1365 3996 50  0000 L CNN
+F 1 "0,1" H 1365 3905 50  0000 L CNN
+F 2 "Capacitors_SMD:C_0603" H 1288 3800 50  0001 C CNN
+F 3 "" H 1250 3950 50  0001 C CNN
+	1    1250 3950
+	-1   0    0    1
+$EndComp
+$Comp
+L device1:C C?
+U 1 1 5A819CD1
+P 1675 3950
+F 0 "C?" H 1790 3996 50  0000 L CNN
+F 1 "0,1" H 1790 3905 50  0000 L CNN
+F 2 "Capacitors_SMD:C_0603" H 1713 3800 50  0001 C CNN
+F 3 "" H 1675 3950 50  0001 C CNN
+	1    1675 3950
+	-1   0    0    1
+$EndComp
+$Comp
+L power1:GND #PWR?
+U 1 1 5A819D53
+P 1675 4100
+F 0 "#PWR?" H 1675 3850 50  0001 C CNN
+F 1 "GND" H 1680 3927 50  0001 C CNN
+F 2 "" H 1675 4100 50  0001 C CNN
+F 3 "" H 1675 4100 50  0001 C CNN
+	1    1675 4100
+	-1   0    0    -1
+$EndComp
+$Comp
+L power1:GND #PWR?
+U 1 1 5A819DBE
+P 1250 4100
+F 0 "#PWR?" H 1250 3850 50  0001 C CNN
+F 1 "GND" H 1255 3927 50  0001 C CNN
+F 2 "" H 1250 4100 50  0001 C CNN
+F 3 "" H 1250 4100 50  0001 C CNN
+	1    1250 4100
+	-1   0    0    -1
+$EndComp
+Text Label 1250 3800 0    60   ~ 0
+VCAP1
+Text Label 1675 3800 0    60   ~ 0
+VCAP2
 $EndSCHEMATC

Commit message: Add I2C pullups
Parts:
- added R? (x2): DNF, Resistors_SMD:R_0603, symbol device1:R
- gave numbers to parts that had none: 2
Connections:
- wire segments 271 -> 280
Changed lines of the file:
@@
 Text GLabel 8750 2825 2    60   Input ~ 0
 +3V3
-Text GLabel 13100 6100 2    50   Output ~ 0
+Text GLabel 13950 6100 2    50   Output ~ 0
 SCL
-Text GLabel 13100 6200 2    50   BiDi ~ 0
+Text GLabel 13950 6200 2    50   BiDi ~ 0
 SDA
 Text Notes 775  5025 0    60   ~ 0
@@
 Text Label 13650 5600 2    60   ~ 0
 LCD_DC
-Text Label 3125 5100 0    60   ~ 0
+Text Label 3825 5100 0    50   ~ 0
 LCD_RESET
-Text Label 13650 6300 2    60   ~ 0
+Text Label 13225 6300 2    50   ~ 0
 BUTTON1
 Text Label 13650 5400 2    60   ~ 0
@@
 	4275 6500 4000 6500
 Wire Wire Line
-	3650 4650 3725 4550
-Wire Wire Line
-	3725 4550 4075 4550
+	3650 4650 3650 4550
+Wire Wire Line
+	3650 4550 4075 4550
 Wire Wire Line
 	4075 4550 4075 4800
@@
 	4275 4900 4075 4900
 Wire Wire Line
-	4075 4900 4075 5025
-Wire Wire Line
-	4075 5025 3725 5025
-Wire Wire Line
-	3725 5025 3650 4950
+	4075 4900 4075 4950
 Wire Wire Line
 	7475 8950 7475 8800
@@
 	8575 2825 8750 2825
 Wire Wire Line
-	12875 6100 13100 6100
-Wire Wire Line
-	12875 6200 13100 6200
-Wire Wire Line
-	4275 5100 3125 5100
+	12875 6100 13400 6100
+Wire Wire Line
+	12875 6200 13700 6200
+Wire Wire Line
+	4275 5100 3825 5100
 Wire Wire Line
 	12875 5600 13650 5600
@@
 Wire Wire Line
 	4450 10750 4900 10750
-Text Notes 13800 5775 0    60   ~ 0
+Text Notes 14725 6975 0    60   ~ 0
 5-way SMD Joystick ALPS SKRHABE010
 $Comp
@@
 Text Label 4900 10750 2    60   ~ 0
 RDY
-Text Label 3750 4550 0    50   ~ 0
+Text Label 4075 4550 2    50   ~ 0
 OSC_IN
-Text Label 3775 5025 0    50   ~ 0
+Text Label 3725 4950 0    50   ~ 0
 OSC_OUT
 Text Label 2900 6700 0    60   ~ 0
@@
 BUTTON5
 Wire Wire Line
-	12875 6300 13650 6300
+	12875 6300 13225 6300
 Text Label 14775 6300 2    60   ~ 0
 BUTTON5
@@
 	3750 11275 3750 11775
 Wire Wire Line
-	12875 6400 13650 6400
-Text Label 13650 6400 2    60   ~ 0
+	12875 6400 13225 6400
+Text Label 13225 6400 2    50   ~ 0
 LED1
 Text Label 3800 4000 0    60   ~ 0
@@
 Connection ~ 3650 4950
 Wire Wire Line
-	3500 4500 3725 4500
-Wire Wire Line
-	3725 4500 3725 4550
-Connection ~ 3725 4550
+	3500 4500 3650 4500
+Wire Wire Line
+	3650 4500 3650 4550
+Connection ~ 3650 4550
 $Comp
 L power1:GND #PWR027
@@
 	-1   0    0    1
 $EndComp
-Text GLabel 13675 7200 2    60   Input ~ 0
+Text GLabel 13825 7075 2    60   Input ~ 0
 +5VDC
 $Comp
@@
 +3V3
 $Comp
-L device1:C C?
+L device1:C C21
 U 1 1 5A819C2F
 P 1250 3950
-F 0 "C?" H 1365 3996 50  0000 L CNN
+F 0 "C21" H 1365 3996 50  0000 L CNN
 F 1 "0,1" H 1365 3905 50  0000 L CNN
 F 2 "Capacitors_SMD:C_0603" H 1288 3800 50  0001 C CNN
@@
 $EndComp
 $Comp
-L device1:C C?
+L device1:C C22
 U 1 1 5A819CD1
 P 1675 3950
-F 0 "C?" H 1790 3996 50  0000 L CNN
+F 0 "C22" H 1790 3996 50  0000 L CNN
 F 1 "0,1" H 1790 3905 50  0000 L CNN
 F 2 "Capacitors_SMD:C_0603" H 1713 3800 50  0001 C CNN
@@
 $EndComp
 $Comp
-L power1:GND #PWR?
+L power1:GND #PWR034
 U 1 1 5A819D53
 P 1675 4100
-F 0 "#PWR?" H 1675 3850 50  0001 C CNN
+F 0 "#PWR034" H 1675 3850 50  0001 C CNN
 F 1 "GND" H 1680 3927 50  0001 C CNN
 F 2 "" H 1675 4100 50  0001 C CNN
@@
 $EndComp
 $Comp
-L power1:GND #PWR?
+L power1:GND #PWR035
 U 1 1 5A819DBE
 P 1250 4100
-F 0 "#PWR?" H 1250 3850 50  0001 C CNN
+F 0 "#PWR035" H 1250 3850 50  0001 C CNN
 F 1 "GND" H 1255 3927 50  0001 C CNN
 F 2 "" H 1250 4100 50  0001 C CNN
@@
 Text Label 1675 3800 0    60   ~ 0
 VCAP2
+Wire Wire Line
+	3650 4950 4075 4950
+Wire Wire Line
+	13825 7075 13675 7075
+Wire Wire Line
+	13675 7075 13675 7200
+$Comp
+L device1:R R?
+U 1 1 5A590DB3
+P 13400 5900
+F 0 "R?" V 13193 5900 50  0000 C CNN
+F 1 "DNF" V 13284 5900 50  0000 C CNN
+F 2 "Resistors_SMD:R_0603" V 13330 5900 50  0001 C CNN
+F 3 "" H 13400 5900 50  0001 C CNN
+	1    13400 5900
+	-1   0    0    1
+$EndComp
+$Comp
+L device1:R R?
+U 1 1 5A590F04
+P 13700 5900
+F 0 "R?" V 13493 5900 50  0000 C CNN
+F 1 "DNF" V 13584 5900 50  0000 C CNN
+F 2 "Resistors_SMD:R_0603" V 13630 5900 50  0001 C CNN
+F 3 "" H 13700 5900 50  0001 C CNN
+	1    13700 5900
+	-1   0    0    1
+$EndComp
+Wire Wire Line
+	13400 6050 13400 6100
+Connection ~ 13400 6100
+Wire Wire Line
+	13400 6100 13950 6100
+Wire Wire Line
+	13700 6050 13700 6200
+Connection ~ 13700 6200
+Wire Wire Line
+	13700 6200 13950 6200
+Wire Wire Line
+	13400 5750 13400 5700
+Wire Wire Line
+	13400 5700 13700 5700
+Wire Wire Line
+	13700 5750 13700 5700
+Connection ~ 13700 5700
+Wire Wire Line
+	13700 5700 13950 5700
+Text GLabel 13950 5700 2    60   Input ~ 0
++3V3
 $EndSCHEMATC

Commit message: Cleanups
Parts:
- added C23, C24: 10u, Capacitors_SMD:C_1210, symbol device1:C
- gave numbers to parts that had none: 2
Connections:
- wire segments 280 -> 284
Changed lines of the file:
@@
 Connection ~ 9925 9000
 Wire Wire Line
-	9925 9000 10325 9000
+	9925 9000 10400 9000
 Text GLabel 8525 9000 0    60   Input ~ 0
 +5VDC
-Text GLabel 10325 9000 2    60   Output ~ 0
+Text GLabel 11475 9000 2    60   Output ~ 0
 +3V3
 $Comp
@@
 	13675 7075 13675 7200
 $Comp
-L device1:R R?
+L device1:R R6
 U 1 1 5A590DB3
 P 13400 5900
-F 0 "R?" V 13193 5900 50  0000 C CNN
+F 0 "R6" V 13193 5900 50  0000 C CNN
 F 1 "DNF" V 13284 5900 50  0000 C CNN
 F 2 "Resistors_SMD:R_0603" V 13330 5900 50  0001 C CNN
@@
 $EndComp
 $Comp
-L device1:R R?
+L device1:R R7
 U 1 1 5A590F04
 P 13700 5900
-F 0 "R?" V 13493 5900 50  0000 C CNN
+F 0 "R7" V 13493 5900 50  0000 C CNN
 F 1 "DNF" V 13584 5900 50  0000 C CNN
 F 2 "Resistors_SMD:R_0603" V 13630 5900 50  0001 C CNN
@@
 Text GLabel 13950 5700 2    60   Input ~ 0
 +3V3
+$Comp
+L device1:C C23
+U 1 1 5A604934
+P 10400 9250
+F 0 "C23" H 10515 9296 50  0000 L CNN
+F 1 "10u" H 10515 9205 50  0000 L CNN
+F 2 "Capacitors_SMD:C_1210" H 10438 9100 50  0001 C CNN
+F 3 "" H 10400 9250 50  0001 C CNN
+	1    10400 9250
+	1    0    0    -1
+$EndComp
+$Comp
+L power1:GND #PWR036
+U 1 1 5A60493A
+P 10400 9400
+F 0 "#PWR036" H 10400 9150 50  0001 C CNN
+F 1 "GND" H 10405 9227 50  0001 C CNN
+F 2 "" H 10400 9400 50  0001 C CNN
+F 3 "" H 10400 9400 50  0001 C CNN
+	1    10400 9400
+	1    0    0    -1
+$EndComp
+Wire Wire Line
+	10400 9100 10400 9000
+Connection ~ 10400 9000
+Wire Wire Line
+	10400 9000 10800 9000
+$Comp
+L device1:C C24
+U 1 1 5A61C13C
+P 10800 9250
+F 0 "C24" H 10915 9296 50  0000 L CNN
+F 1 "10u" H 10915 9205 50  0000 L CNN
+F 2 "Capacitors_SMD:C_1210" H 10838 9100 50  0001 C CNN
+F 3 "" H 10800 9250 50  0001 C CNN
+	1    10800 9250
+	1    0    0    -1
+$EndComp
+$Comp
+L power1:GND #PWR037
+U 1 1 5A61C142
+P 10800 9400
+F 0 "#PWR037" H 10800 9150 50  0001 C CNN
+F 1 "GND" H 10805 9227 50  0001 C CNN
+F 2 "" H 10800 9400 50  0001 C CNN
+F 3 "" H 10800 9400 50  0001 C CNN
+	1    10800 9400
+	1    0    0    -1
+$EndComp
+Wire Wire Line
+	10800 9100 10800 9000
+Connection ~ 10800 9000
+Wire Wire Line
+	10800 9000 11475 9000
 $EndSCHEMATC

Commit message: Schematic cleanup
Connections:
- wire segments 284 -> 283
Other:
- note removed: "BUTTONS, LED(s) and BEEPER"
- note removed: "SN74LV1T34 Logic Buffer Translator\nSN74LVC2G07 Dual Open Drain Buffer"
- note removed: "use open drain"
